File: pcb/Guitar_waveform_proj.kicad_pcb (KiCad board)
At the start: 2 copper layers, 50.5 x 102 mm, 40 parts, among them J1 NMJ6HFD2, J2 NMJ6HFD2, Q1 TP0604, Q2 2N3906, Q3 2N3904, U1 9V Jack, U2 MPM3610, U3 LM324, U4 Huzzah32, U5 Adafruit 1.44" ST7735

Commit message: Added final details about v1.0.0
Updated the notes,
updated the pcb files somewhere I think? Nothing major, just touch ups
Other:
- board text added: "Notes: Mounting holes are sized for M2 screws"
- board text removed: "Notes: Mounting holes are sized for M2 screws The PCB must be mounted before the Huzzah32 is installed. Female pin headers are highly recommended to allow easy installation and disassembly."
Changed lines of the file:
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@@
     (effects (font (size 3 3) (thickness 0.25) bold) (justify left bottom))
   )
-  (gr_text "Notes:\n\nMounting holes are sized for M2 screws\n\nThe PCB must be mounted before the Huzzah32 is installed.\nFemale pin headers are highly recommended to allow easy\ninstallation and disassembly." (at 46.99 56.515) (layer "Cmts.User")
+  (gr_text "Notes:\n\nMounting holes are sized for M2 screws" (at 46.99 56.515) (layer "Cmts.User")
     (effects (font (size 2 2) (thickness 0.25)) (justify left bottom))
   )
